Commit message: update simualtion of ufactorybots

File: simulation/Lite6/lite6.urdf (robot description, URDF)
Before this commit: robot lite6, 8 links, 7 joints
Links:
- added link world
- link link1: geometry collision mesh filename=package://xarm_description/meshes/lite6/collision/link1.stl; visual mesh filename=package://xarm_description/meshes/lite6/visual/link1.stl
- link link2: geometry collision mesh filename=package://xarm_description/meshes/lite6/collision/link2.stl; visual mesh filename=package://xarm_description/meshes/lite6/visual/link2.stl
- link link3: geometry collision mesh filename=package://xarm_description/meshes/lite6/collision/link3.stl; visual mesh filename=package://xarm_description/meshes/lite6/visual/link3.stl
- link link4: geometry collision mesh filename=package://xarm_description/meshes/lite6/collision/link4.stl; visual mesh filename=package://xarm_description/meshes/lite6/visual/link4.stl
- link link5: geometry collision mesh filename=package://xarm_description/meshes/lite6/collision/link5.stl; visual mesh filename=package://xarm_description/meshes/lite6/visual/link5.stl
- link link6: mass 0.180 -> 0.13; geometry collision mesh filename=package://xarm_description/meshes/lite6/collision/link6.stl; visual mesh filename=package://xarm_description/meshes/lite6/visual/link6.stl
- link link_base: mass 2.11 -> 1.65393501783165; geometry collision mesh filename=package://xarm_description/meshes/lite6/collision/link_base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; visual mesh filename=package://xarm_description/meshes/lite6/visual/link_base.stl
Joints:
- added joint world_joint: type fixed, parent world, child link_base, origin xyz=0 0 0 rpy=0 0 0
- joint joint1: limit lower=-6.28 upper=6.28 effort=32.0 velocity=3.14 -> lower=-6.283185307179586 upper=6.283185307179586 effort=50.0 velocity=3.14; origin xyz=0 0 0.2433 rpy=0 0 0 -> xyz=0 0 0.2435 rpy=0 0 0
- joint joint2: limit lower=-2.61799 upper=2.61799 effort=32.0 velocity=3.14 -> lower=-2.61799 upper=2.61799 effort=50.0 velocity=3.14
- joint joint3: limit lower=-0.061087 upper=5.235988 effort=18.0 velocity=3.14 -> lower=-0.061087 upper=5.235988 effort=32.0 velocity=3.14; origin xyz=0.2 0 0 rpy=-3.1416 0 1.5708 -> xyz=0.2002 0 0 rpy=-3.1416 0 1.5708
- joint joint4: limit lower=-6.28 upper=6.28 effort=2.5 velocity=3.14 -> lower=-6.283185307179586 upper=6.283185307179586 effort=32.0 velocity=3.14; origin xyz=0.087 -0.2276 0 rpy=1.5708 0 0 -> xyz=0.087 -0.22761 0 rpy=1.5708 0 0
- joint joint5: limit lower=-2.1642 upper=2.1642 effort=2.5 velocity=3.14 -> lower=-2.1642 upper=2.1642 effort=32.0 velocity=3.14
- joint joint6: limit lower=-6.28 upper=6.28 effort=2.5 velocity=3.14 -> lower=-6.283185307179586 upper=6.283185307179586 effort=20.0 velocity=3.14; origin xyz=0 0.0615 0 rpy=-1.5708 0 0 -> xyz=0 0.0625 0 rpy=-1.5708 0 0
