Commit message: Update URDF file for UF850 robot to use relative mesh paths
- Changed mesh file paths from absolute to relative for better portability.
- Updated visual and collision geometry references for all links in the UF850 model.

File: simulation/uf850/uf850.urdf (robot description, URDF)
Before this commit: robot uf850_robot, 8 links, 7 joints
Links:
- link link1: geometry collision mesh filename=meshes/uf850/collision/link1.stl; visual mesh filename=meshes/uf850/visual/link1.stl
- link link2: geometry collision mesh filename=meshes/uf850/collision/link2.stl; visual mesh filename=meshes/uf850/visual/link2.stl
- link link3: geometry collision mesh filename=meshes/uf850/collision/link3.stl; visual mesh filename=meshes/uf850/visual/link3.stl
- link link4: geometry collision mesh filename=meshes/uf850/collision/link4.stl; visual mesh filename=meshes/uf850/visual/link4.stl
- link link5: geometry collision mesh filename=meshes/uf850/collision/link5.stl; visual mesh filename=meshes/uf850/visual/link5.stl
- link link6: geometry collision mesh filename=meshes/uf850/collision/link6.stl; visual mesh filename=meshes/uf850/visual/link6.stl
- link link_base: geometry collision mesh filename=meshes/uf850/collision/link_base.stl; visual mesh filename=meshes/uf850/visual/link_base.stl
